Commit message: can execute planning

File: config/abb_irb6700_200_260_macro.srdf.xacro (robot description, xacro)
@@ -25,5 +25,5 @@
         <joint name="joint_3" value="0"/>
         <joint name="joint_4" value="0"/>
-        <joint name="joint_5" value="0"/>
+        <joint name="joint_5" value="0.5235988421773261"/>
         <joint name="joint_6" value="0"/>
     </group_state>
